Commit message: Switch to force-based teleop
The velocity based one was doing screwy things to the gazebo physics.

File: segway_description/urdf/RMP_OMNI/rmp.urdf.xacro (robot description, xacro)
@@ -44,16 +44,21 @@
     <xacro:property name="battery_offset" value="0.09298" />
     <xacro:macro name="segway_robot">
-        <!-- Base link is the center of the robot's chassis between the motors -->
-        <link name="base_link"/>
-        <gazebo>
-            <plugin name="gazebo_ros_control" filename="libgazebo_ros_control.so"/>
-            <plugin name="object_controller" filename="libgazebo_ros_planar_move.so">
-                <commandTopic>cmd_vel</commandTopic>
-                <odometryTopic>odom</odometryTopic>
-                <odometryFrame>odom</odometryFrame>
-                <odometryRate>100</odometryRate>
-                <robotBaseFrame>base_link</robotBaseFrame>
-            </plugin>
-        </gazebo>
+    <!-- Base link is the center of the robot's chassis between the motors -->
+    <link name="base_link"/>
+    <gazebo>
+      <plugin name="gazebo_ros_control" filename="libgazebo_ros_control.so"/>
+      <plugin name="ridgeback_ros_force_based_move" filename="libridgeback_ros_force_based_move.so">
+        <commandTopic>cmd_vel</commandTopic>
+        <odometryTopic>odom</odometryTopic>
+        <odometryFrame>odom</odometryFrame>
+        <odometryRate>25.0</odometryRate>
+        <robotBaseFrame>base_link</robotBaseFrame>
+        <cmdVelTimeOut>0.25</cmdVelTimeOut>
+        <publishOdometryTf>0</publishOdometryTf>
+        <yaw_velocity_p_gain>500.0</yaw_velocity_p_gain>
+        <x_velocity_p_gain>10000.0</x_velocity_p_gain>
+        <y_velocity_p_gain>10000.0</y_velocity_p_gain>
+      </plugin>
+    </gazebo>
         <!-- Base footprint is on the ground under the robot -->
         <link name="base_chassis_link"/>
